File: CTRX/CTRX.kicad_sch (KiCad schematic)
At the start: 33 parts, among them J1 CON-SMA-EDGE-S, J3 Conn_02x05_Odd_Even, J4 USB-AM-S-X-X-TH, U1 nRF52820-QDxx, U2 NRF21540-QDAA-R7, U3 USBLC6-2SC6, U4 ME6211C33M5, Y1 32MHz

Commit message: CTRX updated
Parts:
- removed C2: 4.7uF, Capacitor_SMD:C_0603_1608Metric, symbol Device:C_Small
- D1, D2: footprint LED_SMD:LED_0402_1005Metric -> LED_SMD:LED_0805_2012Metric
- L1, L2: footprint Inductor_SMD:L_0201_0603Metric -> Inductor_SMD:L_0402_1005Metric
Other:
- moved on the sheet: C1, C3, C4, C5

Commit message: antenna
Parts:
- added C2: 1pF, Capacitor_SMD:C_0201_0603Metric, symbol Device:C_Small
- added C7: 1.2pF, Capacitor_SMD:C_0201_0603Metric, symbol Device:C_Small
- added L3: 4.7nH, Inductor_SMD:L_0201_0603Metric, symbol Device:L_Small
- added L4: 2.2nH, Inductor_SMD:L_0201_0603Metric, symbol Device:L_Small
- C11, C18, C8: footprint Capacitor_SMD:C_0402_1005Metric -> Capacitor_SMD:C_0201_0603Metric
- C12, C15: value 12pF -> 8pF
- L1, L2: footprint Inductor_SMD:L_0402_1005Metric -> Inductor_SMD:L_0201_0603Metric
Connections:
- net GND: now also C2.2, C7.2
- net NRF_ANT: now also L4.2; no longer U1.24 (ANT)
- new net: C2.1, L3.1, U1.24 (ANT)
- new net: C7.1, L3.2, L4.1
Other:
- moved on the sheet: C10, C13, C14, C6, U1

Commit message: ready
Connections:
- net +3.3V: no longer U1.9 (VDDH)
- net +5V: now also U1.9 (VDDH)
Other:
- moved on the sheet: C10, C13, C14, C6, C9, L2

Commit message: CTRX Order Ready
Parts:
- added C19: 4.7uF, Capacitor_SMD:C_0603_1608Metric, symbol Device:C_Small
Connections:
- net +3.3V: now also C1.2, C3.1, C4.1, C5.1
- net +5V: now also C19.1; no longer C1.2, C3.1, C4.1, C5.1
- net GND: now also C19.2; no longer J3.3 (Pin_3), J3.5 (Pin_5)
- net NRF_SWDIO: now also J3.2 (Pin_2); no longer J3.8 (Pin_8)
- net P014: now also J3.3 (Pin_3); no longer J3.2 (Pin_2)
- net P015: now also J3.5 (Pin_5); no longer J3.6 (Pin_6)
- no-connect marks 8 -> 10
Other:
- moved on the sheet: J3, J4
